File: Capacitance_Meter/Power_Supply.sch (KiCad schematic (older format))
At the start: 5 parts, among them SW1 SW_SPDT

Commit message: USB library and footprint
Parts:
- C1, C2: footprint (none) -> Capacitor_SMD:C_0805_2012Metric
- USB1: footprint (none) -> USB_Connectors:USB_micro_B_female
Changed lines of the file:
@@
 F 0 "USB1" H 4157 3917 50  0000 C CNN
 F 1 "USB_B_Micro" H 4157 3826 50  0000 C CNN
-F 2 "" H 4250 3400 50  0001 C CNN
+F 2 "USB_Connectors:USB_micro_B_female" H 4250 3400 50  0001 C CNN
 F 3 "~" H 4250 3400 50  0001 C CNN
 	1    4100 3450
@@
 F 0 "C1" H 5465 3346 50  0000 L CNN
 F 1 "0.33u" H 5465 3255 50  0000 L CNN
-F 2 "" H 5388 3150 50  0001 C CNN
+F 2 "Capacitor_SMD:C_0805_2012Metric" H 5388 3150 50  0001 C CNN
 F 3 "~" H 5350 3300 50  0001 C CNN
 	1    5350 3300
@@
 F 0 "C2" H 6665 3346 50  0000 L CNN
 F 1 "0.1u" H 6665 3255 50  0000 L CNN
-F 2 "" H 6588 3150 50  0001 C CNN
+F 2 "Capacitor_SMD:C_0805_2012Metric" H 6588 3150 50  0001 C CNN
 F 3 "~" H 6550 3300 50  0001 C CNN
 	1    6550 3300

Commit message: Update to capacitance meter
Parts:
- LDO1: footprint (none) -> Package_TO_SOT_SMD:SOT-89-3
- SW1: footprint (none) -> Switches:Vertical_slide_switch
Changed lines of the file:
@@
 $Descr A4 11693 8268
 encoding utf-8
-Sheet 2 3
+Sheet 2 5
 Title "Capacitance Meter"
 Date "2020-05-24"
@@
 AR Path="/5ECA7B13/5ECB311E" Ref="USB?"  Part="1"
 AR Path="/5ECB157C/5ECB311E" Ref="USB1"  Part="1"
+AR Path="/5EDD65A8/5ECB311E" Ref="USB?"  Part="1"
 F 0 "USB1" H 4157 3917 50  0000 C CNN
 F 1 "USB_B_Micro" H 4157 3826 50  0000 C CNN
@@
 AR Path="/5ECA7B13/5ECB3124" Ref="SW?"  Part="1"
 AR Path="/5ECB157C/5ECB3124" Ref="SW1"  Part="1"
+AR Path="/5EDD65A8/5ECB3124" Ref="SW?"  Part="1"
 F 0 "SW1" H 4800 3535 50  0000 C CNN
 F 1 "SW_SPDT" H 4800 3444 50  0000 C CNN
-F 2 "" H 4800 3250 50  0001 C CNN
+F 2 "Switches:Vertical_slide_switch" H 4800 3250 50  0001 C CNN
 F 3 "~" H 4800 3250 50  0001 C CNN
 	1    4800 3250
@@
 AR Path="/5ECA7B13/5ECB312A" Ref="LDO?"  Part="1"
 AR Path="/5ECB157C/5ECB312A" Ref="LDO1"  Part="1"
+AR Path="/5EDD65A8/5ECB312A" Ref="LDO?"  Part="1"
 F 0 "LDO1" H 5950 3392 50  0000 C CNN
 F 1 "L7805" H 5950 3301 50  0000 C CNN
-F 2 "" H 5975 3000 50  0001 L CIN
+F 2 "Package_TO_SOT_SMD:SOT-89-3" H 5975 3000 50  0001 L CIN
 F 3 "http://www.st.com/content/ccc/resource/technical/document/datasheet/41/4f/b3/b0/12/d4/47/88/CD00000444.pdf/files/CD00000444.pdf/jcr:content/translations/en.CD00000444.pdf" H 5950 3100 50  0001 C CNN
 	1    5950 3150
@@
 AR Path="/5ECA7B13/5ECB3130" Ref="C?"  Part="1"
 AR Path="/5ECB157C/5ECB3130" Ref="C1"  Part="1"
+AR Path="/5EDD65A8/5ECB3130" Ref="C?"  Part="1"
 F 0 "C1" H 5465 3346 50  0000 L CNN
 F 1 "0.33u" H 5465 3255 50  0000 L CNN
@@
 AR Path="/5ECA7B13/5ECB3136" Ref="C?"  Part="1"
 AR Path="/5ECB157C/5ECB3136" Ref="C2"  Part="1"
+AR Path="/5EDD65A8/5ECB3136" Ref="C?"  Part="1"
 F 0 "C2" H 6665 3346 50  0000 L CNN
 F 1 "0.1u" H 6665 3255 50  0000 L CNN
@@
 AR Path="/5ECA7B13/5ECB313C" Ref="#PWR?"  Part="1"
 AR Path="/5ECB157C/5ECB313C" Ref="#PWR0101"  Part="1"
+AR Path="/5EDD65A8/5ECB313C" Ref="#PWR?"  Part="1"
 F 0 "#PWR0101" H 5350 3200 50  0001 C CNN
 F 1 "GND" H 5355 3277 50  0000 C CNN
@@
 AR Path="/5ECA7B13/5ECB3142" Ref="#PWR?"  Part="1"
 AR Path="/5ECB157C/5ECB3142" Ref="#PWR0102"  Part="1"
+AR Path="/5EDD65A8/5ECB3142" Ref="#PWR?"  Part="1"
 F 0 "#PWR0102" H 5950 3200 50  0001 C CNN
 F 1 "GND" H 5955 3277 50  0000 C CNN
@@
 AR Path="/5ECA7B13/5ECB3148" Ref="#PWR?"  Part="1"
 AR Path="/5ECB157C/5ECB3148" Ref="#PWR0103"  Part="1"
+AR Path="/5EDD65A8/5ECB3148" Ref="#PWR?"  Part="1"
 F 0 "#PWR0103" H 6550 3200 50  0001 C CNN
 F 1 "GND" H 6555 3277 50  0000 C CNN
@@
 AR Path="/5ECA7B13/5ECB314E" Ref="#PWR?"  Part="1"
 AR Path="/5ECB157C/5ECB314E" Ref="#PWR0104"  Part="1"
+AR Path="/5EDD65A8/5ECB314E" Ref="#PWR?"  Part="1"
 F 0 "#PWR0104" H 4100 3600 50  0001 C CNN
 F 1 "GND" H 4105 3677 50  0000 C CNN
@@
 U 1 1 5ECABDEA
 P 6900 3150
+AR Path="/5ECB157C/5ECABDEA" Ref="#PWR0105"  Part="1"
+AR Path="/5EDD65A8/5ECABDEA" Ref="#PWR?"  Part="1"
 F 0 "#PWR0105" H 6900 3000 50  0001 C CNN
 F 1 "+3.3V" H 6915 3323 50  0000 C CNN
