File: Capacitance_Meter/Interface.sch (KiCad schematic (older format))
At the start: 2 parts, among them SW2 SW_Push

Commit message: DC load project added
Parts:
- OLED1: symbol Displays:SSD1306_OLED_I2C -> Capacitance_Meter-rescue:SSD1306_OLED_I2C-Displays
Changed lines of the file:
@@
 SDA
 $Comp
-L Displays:SSD1306_OLED_I2C OLED1
+L Capacitance_Meter-rescue:SSD1306_OLED_I2C-Displays OLED1
 U 1 1 5EDD94F4
 P 5350 3750
+AR Path="/5EDD94F4" Ref="OLED1"  Part="1"
+AR Path="/5EDD6869/5EDD94F4" Ref="OLED1"  Part="1"
 F 0 "OLED1" H 5300 4150 50  0000 L CNN
 F 1 "SSD1306_OLED_I2C" H 5100 3400 50  0000 L CNN
